File: console64.kicad_pcb (KiCad board)
At the start: 2 copper layers, 234 x 120 mm, 195 parts, among them IC1 ARD-PRO-MINI-5, IC2 FDS4935A, J1 USB_C_Receptacle_USB2.0, J2 ICD15S13E6GX00LF, J3 DM3AT-SF-PEJM5, J4 AudioJack3, J5 KEYMATRIX_OUT, J6 STM_UART, J7 PS/2 MOUSE, SW1 SW_Push, SW10 SW_Push, SW11 SW_Push, SW12 SW_Push, SW13 SW_Push, SW14 SW_Push, SW15 SW_Push, SW16 SW_Push, SW17 SW_Push, SW18 SW_Push, SW19 SW_Push, SW2 SW_Push, SW20 SW_Push, SW21 SW_Push, SW22 SW_Push, SW23 SW_Push, SW24 SW_Push, SW25 SW_Push, SW26 SW_Push, SW27 SW_Push, SW28 SW_Push, SW29 SW_Push, SW3 SW_Push, SW30 SW_Push, SW31 SW_Push, SW32 SW_Push, SW33 SW_Push, SW34 SW_Push, SW35 SW_Push, SW36 SW_Push, SW37 SW_Push, SW38 SW_Push, SW39 SW_Push, SW4 SW_Push, SW40 SW_Push, SW41 SW_Push, SW42 SW_Push, SW43 SW_Push, SW44 SW_Push, SW45 SW_Push, SW46 SW_Push, SW47 SW_Push, SW48 SW_Push, SW49 SW_Push, SW5 SW_Push, SW50 SW_Push, SW51 SW_Push, SW52 SW_Push, SW53 SW_Push, SW54 SW_Push, SW55 SW_Push, SW56 SW_Push, SW57 SW_Push, SW58 SW_Push, SW59 SW_Push, SW6 SW_Push, SW60 SW_Push, SW61 SW_Push, SW62 SW_Push, SW63 SW_Push, SW64 SW_Push, SW65 PS-85S, SW7 SW_Push, SW8 SW_Push, SW9 SW_Push, U1 BluePill_1, U2 ESP32-DEVKITC-32D

Commit message: routed
Routing:
- net GND: track 0.00 -> 457.4 mm
- net key_row3: track 0.00 -> 336.1 mm
- net key_row4: track 0.00 -> 333.2 mm
- net key_row2: track 0.00 -> 325.2 mm
- net key_col0: track 0.00 -> 318.4 mm
- net key_row1: track 0.00 -> 315.5 mm
- net key_row0: track 0.00 -> 298.0 mm
- net 5V_ESP: track 0.00 -> 271.1 mm, vias 0 -> 3
- net key_col1: track 0.00 -> 266.2 mm
- net key_col2: track 0.00 -> 263.0 mm
- net key_col3: track 0.00 -> 239.5 mm, vias 0 -> 1
- net key_col4: track 0.00 -> 217.9 mm
- net /61: track 0.00 -> 208.7 mm
- net key_col5: track 0.00 -> 200.4 mm
- net STM_TX: track 0.00 -> 200.4 mm, vias 0 -> 1
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
Commit message: production
Parts:
- added G***: LOGO, bongorian:hardcore, F.Cu at (66.0, 45.0)
- added G***: LOGO, bongorian:c64_back, B.Cu at (147.0, 105.0)
- SW1, SW10, SW11, SW12, SW13, SW14, SW15, SW16, SW17, SW18, SW19, SW2, SW20, SW21, SW22, SW23, SW24, SW25, SW26, SW27, SW28, SW29, SW3, SW30, SW31, SW32, SW33, SW34, SW35, SW36, SW37, SW38, SW39, SW4, SW40, SW41, SW42, SW43, SW44, SW45, SW46, SW47, SW48, SW49, SW5, SW50, SW51, SW52, SW53, SW54, SW55, SW56, SW57, SW58, SW59, SW6, SW60, SW61, SW62, SW63, SW64, SW7, SW8, SW9: footprint bongorian:SW_PG1350_inname -> bongorian:SW_PG1350_inname_ana
Routing:
- net GND: vias 0 -> 56
- added copper zone on B.Cu, net GND
- added copper zone on F.Cu, net GND
